File: Daughterboard (Cantaloupe)/Daughterboard (Cantaloupe).kicad_sch (KiCad schematic)
At the start: 55 parts, among them J3 Pogo, SW1 MX/Choc, SW10 MX/Choc, SW11 MX/Choc, SW12 MX/Choc, SW13 MX/Choc, SW14 MX/Choc, SW15 MX/Choc, SW16 MX/Choc, SW17 MX/Choc, SW18 MX/Choc, SW19 MX/Choc, SW2 MX/Choc, SW20 MX/Choc, SW21 MX/Choc, SW22 MX/Choc, SW23 MX/Choc, SW24 MX/Choc, SW25 MX/Choc, SW26 MX/Choc, SW27 MX/Choc, SW28 MX/Choc, SW29 MX/Choc, SW3 MX/Choc, SW30 MX/Choc, SW31 MX/Choc, SW4 MX/Choc, SW5 MX/Choc, SW6 MX/Choc, SW7 MX/Choc, SW8 MX/Choc, SW9 MX/Choc, U1 74HC595, U2 74HC595, U3 74HC595, U4 74HC595

Commit message: 2026/09/30: V0.4 motherboard update complete
Removed guard ring around the edge of the board. Moved reset button and pogo header down the board. Increased length back to 50mm to allow for an E73-2G4M08S1C version to be developed if desired. Simplified reset circuit - doesn't use the Acheron version anymore. Reduced number of pins in pogo header, as the largest available ones are 2x06. Pinout of pogo header changed to greatly simplify routing - no longer VIK-compliant. Signalis reference and Paw-Connect added back. Changed file structure.
Parts:
- removed D12, D13: ESD441, GB-Package:X1SON_0.6x1mm_P0.65mm_Texas_DPY0002A, symbol GB-Device:D_Polarized_TVS_Small
- removed D14, D15: ESD321, GB-Package:X1SON_0.6x1mm_P0.65mm_Texas_DPY0002A, symbol GB-Device:D_Polarized_TVS_Small
- removed J3: Pogo, GB-Header:PinHeader_2x08_2.54mm_MillMax_PogoPin_823-22-016-10-002101_Double_Sided, symbol Connector_Generic:Conn_02x08_Odd_Even
- added J1: Pogo, GB-Header:PinHeader_2x06_2.54mm_MillMax_PogoPin_823-22-012-10-000101-Double_Sided, symbol Connector_Generic:Conn_02x06_Odd_Even
- D1, D10, D2, D4, D5, D6, D7, D8, D9: value ESD441 -> ESD321; LCSC C53161160 -> C2868952; MPN ESD441DPYR -> ESD321DPYR; Rating (none) -> 4V5 breakdown
- D11: Rating (none) -> 7V breakdown
- D3: Rating (none) -> 4V5 breakdown
- SW1, SW10, SW11, SW12, SW13, SW14, SW15, SW16, SW17, SW18, SW19, SW2, SW20, SW21, SW22, SW23, SW24, SW25, SW26, SW27, SW28, SW29, SW3, SW30, SW31, SW4, SW5, SW6, SW7, SW8, SW9: footprint GB-Switch:SW_MX-Choc_1U_Hotswap_Flippable -> GB-Switch:SW_KB_Choc-KS33_1U_Hotswap_Reversible
Connections:
- net GPIO is gone; now on net SPI_CS: D7.1 (K)
- net I2C_SDA is gone; now on net GPIO4: D4.1 (K)
- net RST is gone; now on net GPIO1: D1.1 (K)
- net +3V3: no longer D3.1 (K)
- net +5V: now also J1.10 (Pin_10)
- net EP: now also J1.12 (Pin_12)
- net GPIO1: now also J1.1 (Pin_1); no longer D6.1 (K)
- net GPIO3: now also D3.1 (K), J1.5 (Pin_5); no longer D2.1 (K)
- net GPIO4: now also J1.7 (Pin_7); no longer D10.1 (K)
- net GPIO5: now also D5.1 (K), SW16.1 (A), SW17.1 (A), SW18.1 (A), SW19.1 (A), SW26.1 (A), SW27.1 (A), SW28.1 (A), SW29.1 (A), SW6.1 (A), SW7.1 (A), SW8.1 (A), SW9.1 (A), J1.9 (Pin_9); no longer D9.1 (K), SW16.2 (B), SW17.2 (B), SW18.2 (B), SW19.2 (B), SW26.2 (B), SW27.2 (B), SW28.2 (B), SW29.2 (B), SW6.2 (B), SW7.2 (B), SW8.2 (B), SW9.2 (B)
- net K04: now also SW6.2 (B), U1.7 (QH); no longer SW6.1 (A), U1.4 (QE)
- net K05: now also SW7.2 (B), U1.6 (QG); no longer SW7.1 (A), U1.5 (QF)
- net K06: now also SW8.2 (B), U1.5 (QF); no longer SW8.1 (A), U1.6 (QG)
- net K07: now also SW9.2 (B), U1.4 (QE); no longer SW9.1 (A), U1.7 (QH)
- net K14: now also SW16.2 (B), U2.7 (QH); no longer SW16.1 (A), U2.4 (QE)
- net K15: now also SW17.2 (B), U2.6 (QG); no longer SW17.1 (A), U2.5 (QF)
- net K16: now also SW18.2 (B), U2.5 (QF); no longer SW19.1 (A), U2.6 (QG)
- net K17: now also SW19.2 (B), U2.4 (QE); no longer SW18.1 (A), U2.7 (QH)
- net K24: now also SW26.2 (B), U3.7 (QH); no longer SW26.1 (A), U3.4 (QE)
- net K25: now also SW27.2 (B), U3.6 (QG); no longer SW27.1 (A), U3.5 (QF)
- net K26: now also SW28.2 (B), U3.5 (QF); no longer SW28.1 (A), U3.6 (QG)
- net K27: now also SW29.2 (B), U3.4 (QE); no longer SW29.1 (A), U3.7 (QH)
- net K34: now also U4.7 (QH); no longer U4.4 (QE)
- net K35: now also U4.6 (QG); no longer U4.5 (QF)
- net K36: now also U4.5 (QF); no longer U4.6 (QG)
- net K37: now also U4.4 (QE); no longer U4.7 (QH)
- net RGB_DAT: no longer D5.1 (K)
- net SPI_CS: now also J1.2 (Pin_2)
- net SPI_MISO: now also D10.1 (K), J1.8 (Pin_8); no longer D8.1 (K)
- net SPI_MOSI: now also D9.1 (K), J1.6 (Pin_6)
- net SPI_SCK: now also D8.1 (K), J1.4 (Pin_4)
- new net GPIO2: D2.1 (K), J1.3 (Pin_3)
- new net VDD: D6.1 (K), J1.11 (Pin_11)
Other:
- note removed: "3V6 tolerant only"

Commit message: 2026/10/01: Changed library name and updated paths
Parts:
- C1, C2, C3, C4: footprint GB-Device:C_0402_1005Metric -> Kaleidogeist-Device:C_0402_1005Metric
- D1, D10, D11, D2, D3, D4, D5, D6, D7, D8, D9: footprint GB-Package:X1SON_0.6x1mm_P0.65mm_Texas_DPY0002A -> Kaleidogeist-Package:X1SON_0.6x1mm_P0.65mm_Texas_DPY0002A; symbol GB-Device:D_Polarized_TVS_Small -> Kaleidogeist-Device:D_Polarized_TVS_Small
- J1: footprint GB-Header:PinHeader_2x06_2.54mm_MillMax_PogoPin_823-22-012-10-000101-Double_Sided -> Kaleidogeist-Header:PinHeader_2x06_2.54mm_MillMax_PogoPin_823-22-012-10-000101-Double_Sided
- SW1, SW10, SW11, SW12, SW13, SW14, SW15, SW16, SW17, SW18, SW19, SW2, SW20, SW21, SW22, SW23, SW24, SW25, SW26, SW27, SW28, SW29, SW3, SW30, SW31, SW4, SW5, SW6, SW7, SW8, SW9: footprint GB-Switch:SW_KB_Choc-KS33_1U_Hotswap_Reversible -> Kaleidogeist-Switch:SW_KB_Choc-KS33_1U_Hotswap_Reversible; symbol GB-Switch:SW_Push_Small -> Kaleidogeist-Switch:SW_Push_Small
- U1, U2, U3, U4: footprint GB-Package:DHVQFN-16-1EP_2.5x3.5mm_P0.5mm_EP1x2mm -> Kaleidogeist-Package:DHVQFN-16-1EP_2.5x3.5mm_P0.5mm_EP1x2mm; symbol GB-IC:74HC595B -> Kaleidogeist-IC:74HC595B
