File: Motherboard (G0B1)/Motherboard (G0B1).kicad_sch (KiCad schematic)
At the start: 66 parts, among them J1 USB-C In, J2 USB-C Split, J3 Pogo, J4 SWD, Q1 2N7002W, SW1 Reset, U1 TPD4E05U06, U2 STM32G0B1CCU7, U3 TPS2553-1, U4 XC6206P332MR, U5 TPS2553-1, U6 TPD4E05U06

Commit message: 2026/10/01: Changed library name and updated paths
Parts:
- C1, C10, C3, C4, C6, C7, C8: footprint GB-Device:C_0402_1005Metric -> Kaleidogeist-Device:C_0402_1005Metric
- C11, C12, C2, C5, C9: footprint GB-Device:C_0603_1608Metric -> Kaleidogeist-Device:C_0603_1608Metric
- D1, D10, D11, D12, D13, D2, D3, D4, D5, D6, D7, D8, D9: footprint GB-Package:X1SON_0.6x1mm_P0.65mm_Texas_DPY0002A -> Kaleidogeist-Package:X1SON_0.6x1mm_P0.65mm_Texas_DPY0002A; symbol GB-Device:D_Polarized_TVS_Small -> Kaleidogeist-Device:D_Polarized_TVS_Small
- FB1, FB2, FB3: footprint GB-Device:L_0402_1005Metric -> Kaleidogeist-Device:L_0402_1005Metric
- H1, H2: footprint GB-HolePad:MountingHole_3.2mm_M3_Pad_Via -> Kaleidogeist-HolePad:MountingHole_3.2mm_M3_Pad_Via; symbol GB-Misc:MountingHole_Pad -> Kaleidogeist-Misc:MountingHole_Pad
- J1, J2: footprint GB-Connector:USB_C_Receptacle_Molex_2169900001 -> Kaleidogeist-Connector:USB_C_Receptacle_Molex_2169900001
- J3: footprint GB-Header:PinHeader_2x06_2.54mm_MillMax_PogoTarget_419-10-212-00-001000-Double_Sided -> Kaleidogeist-Header:PinHeader_2x06_2.54mm_MillMax_PogoTarget_419-10-212-00-001000-Double_Sided
- JP1: footprint GB-Misc:SolderJumper-2_P1.2mm_Open_Pad1.0x1.4mm -> Kaleidogeist-Misc:SolderJumper-2_P1.2mm_Open_Pad1.0x1.4mm; symbol GB-Misc:SolderJumper_2_Open -> Kaleidogeist-Misc:SolderJumper_2_Open
- Q1: footprint GB-Package:SOT-323_SC-70-3 -> Kaleidogeist-Package:SOT-323_SC-70-3
- R10, R11, R12, R15, R16, R18, R19, R2, R22, R23, R24, R25, R26, R3, R4, R5, R6, R7, R8, R9: footprint GB-Device:R_0402_1005Metric -> Kaleidogeist-Device:R_0402_1005Metric
- SW1: footprint GB-Switch:SW_Alps_SKSNLM_SKSNLP -> Kaleidogeist-Switch:SW_Alps_SKSNLM_SKSNLP; symbol GB-Switch:SW_Push_Small_MP -> Kaleidogeist-Switch:SW_Push_Small_MP
- TOOL1, TOOL2, TOOL3: footprint GB-HolePad:MountingHole_JLC-Tooling -> Kaleidogeist-HolePad:MountingHole_JLC-Tooling
- U1, U6: footprint GB-Package:USON-10_2.5x1.0mm_P0.5mm -> Kaleidogeist-Package:USON-10_2.5x1.0mm_P0.5mm; symbol GB-IC:TPD4E05U06 -> Kaleidogeist-IC:TPD4E05U06
- U2: footprint GB-Package:QFN-48-1EP_7x7mm_P0.5mm_EP5.6x5.6mm -> Kaleidogeist-Package:QFN-48-1EP_7x7mm_P0.5mm_EP5.6x5.6mm
- U3, U5: footprint GB-Package:WSON-6-1EP_2x2mm_P0.65mm_EP1x1.6mm -> Kaleidogeist-Package:WSON-6-1EP_2x2mm_P0.65mm_EP1x1.6mm; symbol GB-IC:TPS2553DR -> Kaleidogeist-IC:TPS2553DR
- U4: footprint GB-Package:SOT-23-3 -> Kaleidogeist-Package:SOT-23-3
Other:
- company: By Ghostly Butterfly (https://github.com/ghostlybutterfly/Galia/) -> By Kaleidogeist (https://github.com/Kaleidogeist/Galia/)
